File: src/UartFEC.kicad_pcb (KiCad board)
At the start: 2 copper layers, 24 x 27.9 mm, 20 parts, among them J1 B3B-XH-A, P1 105444-0001, Q1 DMP3099L-13, U1 FT232RL

Commit message: Refactoring copper pour
Routing:
- net GND: track 123.1 -> 133.0 mm, vias 7 -> 8
Other:
- rule pad_to_mask_clearance: 0 -> 0.05
Changed lines of the file:
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@@
       (dielectric_constraints no)
     )
-    (pad_to_mask_clearance 0)
+    (pad_to_mask_clearance 0.05)
     (aux_axis_origin 20 20)
     (pcbplotparams
@@
     (at 40.4 35 180)
     (attr smd)
-    (fp_text reference "Q1" (at 1.2 -1.5) (layer "F.SilkS")
+    (fp_text reference "Q1" (at -1.2 -1.5) (layer "F.SilkS")
         (effects (font (size 0.8 0.6) (thickness 0.15)))
     )
@@
     (fp_rect (start -1.35 -0.25) (end 1.35 0.25)
       (stroke (width 0.2) (type default)) (fill none) (layer "F.SilkS"))
-    (fp_circle (center -1.575 1.15) (end -1.425 1.15)
+    (fp_circle (center -1.65 1.15) (end -1.5 1.15)
       (stroke (width 0.1) (type solid)) (fill solid) (layer "F.SilkS"))
     (fp_rect (start -1.75 -1.95) (end 1.75 1.95)
@@
   (segment (start 29.925 29.1) (end 33 29.1) (width 0.25) (layer "F.Cu") (net 7))
   (segment (start 34.75 22.95697) (end 34.75 22.1) (width 0.2) (layer "F.Cu") (net 7))
+  (segment (start 33.075 29.725) (end 30.5 32.3) (width 0.2) (layer "F.Cu") (net 7))
   (segment (start 33.125 29.725) (end 33.1 29.7) (width 0.2) (layer "F.Cu") (net 7))
   (segment (start 27 32.2) (end 27 31.6) (width 0.25) (layer "F.Cu") (net 7))
@@
   (segment (start 42.3 24.8) (end 41.4 25.7) (width 0.25) (layer "F.Cu") (net 7))
   (segment (start 35.5 29.725) (end 33.125 29.725) (width 0.2) (layer "F.Cu") (net 7))
+  (segment (start 30.5 32.3) (end 30.5 35) (width 0.2) (layer "F.Cu") (net 7))
   (segment (start 27.325 29.075) (end 28.5 29.075) (width 0.25) (layer "F.Cu") (net 7))
   (segment (start 27 30.4) (end 27 29.4) (width 0.25) (layer "F.Cu") (net 7))
@@
   (segment (start 32 35.825) (end 32 34.9) (width 0.25) (layer "F.Cu") (net 7))
   (segment (start 28.5 32.325) (end 27.125 32.325) (width 0.25) (layer "F.Cu") (net 7))
+  (segment (start 30.5 35) (end 29.7 35.8) (width 0.2) (layer "F.Cu") (net 7))
+  (segment (start 35.5 29.725) (end 33.075 29.725) (width 0.2) (layer "F.Cu") (net 7))
   (via (at 25.7 31.5) (size 0.6) (drill 0.3) (layers "F.Cu" "B.Cu") (net 7))
   (via (at 32 34.9) (size 0.6) (drill 0.3) (layers "F.Cu" "B.Cu") (net 7))
@@
   (via (at 22.7 45) (size 0.6) (drill 0.3) (layers "F.Cu" "B.Cu") (net 7))
   (via (at 26.9 24.8) (size 0.6) (drill 0.3) (layers "F.Cu" "B.Cu") (net 7))
+  (via (at 29.7 35.8) (size 0.6) (drill 0.3) (layers "F.Cu" "B.Cu") (net 7))
   (segment (start 29.942136 23.742136) (end 34.057864 23.742136) (width 0.2) (layer "B.Cu") (net 7))
   (segment (start 27.8 29.4) (end 25.7 31.5) (width 0.2) (layer "B.Cu") (net 7))
@@
   (via (at 21.5 46.5) (size 0.6) (drill 0.3) (layers "F.Cu" "B.Cu") (net 13))
   (segment (start 21.5 46.5) (end 22.7 46.5) (width 0.2) (layer "B.Cu") (net 13))
-  (segment (start 29.9 34.05) (end 29.9 31.677814) (width 0.2) (layer "F.Cu") (net 14))
-  (segment (start 26 37.95) (end 29.9 34.05) (width 0.2) (layer "F.Cu") (net 14))
+  (segment (start 26 46.5) (end 26 37.95) (width 0.2) (layer "F.Cu") (net 14))
+  (segment (start 31.1 30.477814) (end 31.1 30) (width 0.2) (layer "F.Cu") (net 14))
   (segment (start 31.1 30) (end 30.825 29.725) (width 0.2) (layer "F.Cu") (net 14))
+  (segment (start 30 33.95) (end 30 31.577814) (width 0.2) (layer "F.Cu") (net 14))
   (segment (start 30.825 29.725) (end 28.5 29.725) (width 0.2) (layer "F.Cu") (net 14))
-  (segment (start 29.9 31.677814) (end 31.1 30.477814) (width 0.2) (layer "F.Cu") (net 14))
-  (segment (start 31.1 30.477814) (end 31.1 30) (width 0.2) (layer "F.Cu") (net 14))
-  (segment (start 26 46.5) (end 26 37.95) (width 0.2) (layer "F.Cu") (net 14))
+  (segment (start 26 37.95) (end 30 33.95) (width 0.2) (layer "F.Cu") (net 14))
+  (segment (start 30 31.577814) (end 31.1 30.477814) (width 0.2) (layer "F.Cu") (net 14))
   (via (at 26 46.5) (size 0.6) (drill 0.3) (layers "F.Cu" "B.Cu") (net 14))
   (segment (start 24.5 46.5) (end 26 46.5) (width 0.2) (layer "B.Cu") (net 14))
@@
   (segment (start 41.4 33.8) (end 41.4 31.35) (width 0.2) (layer "F.Cu") (net 17))
   (zone (net 7) (net_name "GND") (layers "F&B.Cu") (hatch edge 0.5)
-    (connect_pads (clearance 0.25))
-    (min_thickness 0.25) (filled_areas_thickness no)
+    (connect_pads no (clearance 0.3))
+    (min_thickness 0.3) (filled_areas_thickness no)
     (fill yes (thermal_gap 0.5) (thermal_bridge_width 0.5))
     (polygon

Commit message: Moved LEDs a bit
Parts:
- moved R1 2.24 mm to (24.0, 44.3)
- moved R2 2.24 mm to (40.0, 44.3)
- moved DS2 1.30 mm to (41.7, 46.5)
- moved DS1 1.30 mm to (22.3, 46.5), turned to 0 degrees
Routing:
- net GND: track 133.0 -> 127.4 mm
- net 5V_SW: track 36.0 -> 31.5 mm
- net LED_RXD: track 22.8 -> 25.2 mm
- net LED_TXD': track 2.35 -> 3.38 mm
- net LED_TXD: track 26.7 -> 27.5 mm

Commit message: Moved LEDs
Parts:
- moved DS1 2.50 mm to (24.8, 46.5)
- moved DS2 2.50 mm to (39.2, 46.5)
Routing:
- net LED_RXD': track 2.26 -> 4.30 mm
- net LED_TXD': track 3.38 -> 4.52 mm
- net LED_RXD: track 25.2 -> 26.1 mm
Changed lines of the file:
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@@
   )
   (footprint "Medo64:DS (0805)" (layer "B.Cu")
-    (at 41.7 46.5)
+    (at 39.2 46.5)
     (descr "LEDC2013X120N")
     (attr smd)
@@
   )
   (footprint "Medo64:DS (0805)" (layer "B.Cu")
-    (at 22.3 46.5)
+    (at 24.8 46.5)
     (descr "LEDC2013X120N")
     (attr smd)
@@
   (segment (start 28.5 30.375) (end 30.375004 30.375) (width 0.2) (layer "F.Cu") (net 11))
   (via (at 30.4 30.399996) (size 0.6) (drill 0.3) (layers "F.Cu" "B.Cu") (net 11))
+  (segment (start 38.3 46.5) (end 38.3 46.3) (width 0.2) (layer "B.Cu") (net 11))
   (segment (start 39.5 30.699992) (end 39.200004 30.399996) (width 0.2) (layer "B.Cu") (net 11))
-  (segment (start 40.8 46.3) (end 39.5 45) (width 0.2) (layer "B.Cu") (net 11))
-  (segment (start 39.5 45) (end 39.5 30.699992) (width 0.2) (layer "B.Cu") (net 11))
-  (segment (start 40.8 46.5) (end 40.8 46.3) (width 0.2) (layer "B.Cu") (net 11))
+  (segment (start 38.3 46.3) (end 39.5 45.1) (width 0.2) (layer "B.Cu") (net 11))
   (segment (start 39.200004 30.399996) (end 30.4 30.399996) (width 0.2) (layer "B.Cu") (net 11))
+  (segment (start 39.5 45.1) (end 39.5 30.699992) (width 0.2) (layer "B.Cu") (net 11))
   (segment (start 40.95 44.3) (end 41.800004 44.3) (width 0.2) (layer "F.Cu") (net 12))
   (via (at 41.800004 44.3) (size 0.6) (drill 0.3) (layers "F.Cu" "B.Cu") (net 12))
-  (segment (start 42.6 45.099996) (end 41.800004 44.3) (width 0.2) (layer "B.Cu") (net 12))
-  (segment (start 42.6 46.5) (end 42.6 45.099996) (width 0.2) (layer "B.Cu") (net 12))
+  (segment (start 40.5 44.3) (end 41.800004 44.3) (width 0.2) (layer "B.Cu") (net 12))
+  (segment (start 40.1 44.7) (end 40.5 44.3) (width 0.2) (layer "B.Cu") (net 12))
+  (segment (start 40.1 46.5) (end 40.1 44.7) (width 0.2) (layer "B.Cu") (net 12))
   (segment (start 23.05 44.3) (end 23.1 44.35) (width 0.2) (layer "F.Cu") (net 13))
   (segment (start 23.1 44.35) (end 23.1 45.415749) (width 0.2) (layer "F.Cu") (net 13))
   (via (at 23.1 45.415749) (size 0.6) (drill 0.3) (layers "F.Cu" "B.Cu") (net 13))
-  (segment (start 23.2 46.5) (end 23.2 45.515749) (width 0.2) (layer "B.Cu") (net 13))
-  (segment (start 23.2 45.515749) (end 23.1 45.415749) (width 0.2) (layer "B.Cu") (net 13))
+  (segment (start 25.7 46.3) (end 24.815749 45.415749) (width 0.2) (layer "B.Cu") (net 13))
+  (segment (start 25.7 46.5) (end 25.7 46.3) (width 0.2) (layer "B.Cu") (net 13))
+  (segment (start 24.815749 45.415749) (end 23.1 45.415749) (width 0.2) (layer "B.Cu") (net 13))
   (segment (start 28.5 29.725) (end 30.825 29.725) (width 0.2) (layer "F.Cu") (net 14))
   (segment (start 31.1 30.477814) (end 30 31.577814) (width 0.2) (layer "F.Cu") (net 14))
@@
   (via (at 26.200009 44.399991) (size 0.6) (drill 0.3) (layers "F.Cu" "B.Cu") (net 14))
   (segment (start 22.800009 44.399991) (end 26.200009 44.399991) (width 0.2) (layer "B.Cu") (net 14))
-  (segment (start 21.4 45.8) (end 22.800009 44.399991) (width 0.2) (layer "B.Cu") (net 14))
-  (segment (start 21.4 46.5) (end 21.4 45.8) (width 0.2) (layer "B.Cu") (net 14))
+  (segment (start 22.4 46.2) (end 22.7 46.5) (width 0.2) (layer "B.Cu") (net 14))
+  (segment (start 22.7 46.5) (end 23.9 46.5) (width 0.2) (layer "B.Cu") (net 14))
+  (segment (start 22.4 44.8) (end 22.800009 44.399991) (width 0.2) (layer "B.Cu") (net 14))
+  (segment (start 22.4 46.2) (end 22.4 44.8) (width 0.2) (layer "B.Cu") (net 14))
   (segment (start 38.29 28.29) (end 36.75 26.75) (width 0.2) (layer "F.Cu") (net 15))
   (segment (start 36.475 25.175) (end 35.5 25.175) (width 0.2) (layer "F.Cu") (net 15))

Commit message: Updated connector designators
Parts:
- renumbered P1 to J1, J1 to J2
Changed lines of the file:
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@@
     (descr "Molex 1054440001")
     (attr smd)
-    (fp_text reference "P1" (at 0 -1.7) (layer "F.SilkS") hide
+    (fp_text reference "J1" (at 0 -1.7) (layer "F.SilkS") hide
         (effects (font (size 0.8 0.6) (thickness 0.15)))
     )
@@
     (descr "JST B3B-XH-A [455-B3B-XH-A-ND]")
     (attr through_hole)
-    (fp_text reference "J1" (at 0 2.9) (layer "F.SilkS")
-        (effects (font (size 0.8 0.6) (thickness 0.15) bold))
-    )
+    (fp_text reference "J2" (at 0 2.9) (layer "F.SilkS")
+        (effects (font (size 0.8 0.6) (thickness 0.15) bold))
+    )

Commit message: Fixed refdes
Parts:
- renumbered C5 to C4, C4 to C5
Changed lines of the file:
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@@
     (tags "CAPC2013X140N")
     (attr smd)
-    (fp_text reference "C5" (at 0 -1.6 90) (layer "F.SilkS") hide
+    (fp_text reference "C4" (at 0 -1.6 90) (layer "F.SilkS") hide
         (effects (font (size 0.8 0.6) (thickness 0.15) bold))
     )
@@
     (tags "CAPC2013X140N")
     (attr smd)
-    (fp_text reference "C4" (at 0 -1.6 90) (layer "F.SilkS") hide
+    (fp_text reference "C5" (at 0 -1.6 90) (layer "F.SilkS") hide
         (effects (font (size 0.8 0.6) (thickness 0.15) bold))
     )
